File: KiCad/KiCad.kicad_pcb (KiCad board)
At the start: 2 copper layers, 76.2 x 76.2 mm, 21 parts, among them J2 Conn_01x04, SW1 SW_Push, U1 ESP32-S3-WROOM-1

Commit message: CHG: minor changes to PCB
Parts:
- turned D1 to 0 degrees
- turned D2 to 0 degrees
- turned D3 to 0 degrees
Routing:
- net GND: track 70.4 -> 55.2 mm
- net Net-(D1-DIN): track 6.07 -> 0.00 mm
- net Net-(D1-VSS): track 5.85 -> 0.00 mm
Changed lines of the file:
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@@
   (net 49 "unconnected-(U1-U0TXD{slash}GPIO43{slash}CLK_OUT1-Pad37)")
   (footprint "LED_SMD:LED_WS2812B_PLCC4_5.0x5.0mm_P3.2mm" (layer "F.Cu")
-    (at 193.04 98.17 90)
+    (at 193.04 98.17)
     (descr "5.0mm x 5.0mm Addressable RGB LED NeoPixel, https://cdn-shop.adafruit.com/datasheets/WS2812B.pdf")
     (tags "LED RGB NeoPixel PLCC-4 5050")
@@
     (property "ki_keywords" "RGB LED NeoPixel addressable")
     (attr smd)
-    (fp_text reference "D3" (at 0 -3.5 90) (layer "F.SilkS")
-        (effects (font (size 1 1) (thickness 0.15)))
-    )
-    (fp_text value "WS2812B" (at 0 4 90) (layer "F.Fab")
-        (effects (font (size 1 1) (thickness 0.15)))
-    )
-    (fp_text user "1" (at -4.15 -1.6 90) (layer "F.SilkS")
-        (effects (font (size 1 1) (thickness 0.15)))
-    )
-    (fp_text user "${REFERENCE}" (at 0 0 90) (layer "F.Fab")
+    (fp_text reference "D3" (at 0 -3.5) (layer "F.SilkS")
+        (effects (font (size 1 1) (thickness 0.15)))
+    )
+    (fp_text value "WS2812B" (at 0 4) (layer "F.Fab")
+        (effects (font (size 1 1) (thickness 0.15)))
+    )
+    (fp_text user "1" (at -4.15 -1.6) (layer "F.SilkS")
+        (effects (font (size 1 1) (thickness 0.15)))
+    )
+    (fp_text user "${REFERENCE}" (at 0 0) (layer "F.Fab")
         (effects (font (size 0.8 0.8) (thickness 0.15)))
     )
@@
     (fp_circle (center 0 0) (end 0 -2)
       (stroke (width 0.1) (type solid)) (fill none) (layer "F.Fab"))
-    (pad "1" smd rect (at -2.45 -1.65 90) (size 1.5 0.9) (layers "F.Cu" "F.Paste" "F.Mask")
+    (pad "1" smd rect (at -2.45 -1.65) (size 1.5 0.9) (layers "F.Cu" "F.Paste" "F.Mask")
       (net 1 "GND") (pinfunction "VDD") (pintype "power_in"))
-    (pad "2" smd rect (at -2.45 1.65 90) (size 1.5 0.9) (layers "F.Cu" "F.Paste" "F.Mask")
+    (pad "2" smd rect (at -2.45 1.65) (size 1.5 0.9) (layers "F.Cu" "F.Paste" "F.Mask")
       (net 6 "Net-(D3-DOUT)") (pinfunction "DOUT") (pintype "output"))
-    (pad "3" smd rect (at 2.45 1.65 90) (size 1.5 0.9) (layers "F.Cu" "F.Paste" "F.Mask")
+    (pad "3" smd rect (at 2.45 1.65) (size 1.5 0.9) (layers "F.Cu" "F.Paste" "F.Mask")
       (net 2 "Net-(D1-VSS)") (pinfunction "VSS") (pintype "power_in"))
-    (pad "4" smd rect (at 2.45 -1.65 90) (size 1.5 0.9) (layers "F.Cu" "F.Paste" "F.Mask")
+    (pad "4" smd rect (at 2.45 -1.65) (size 1.5 0.9) (layers "F.Cu" "F.Paste" "F.Mask")
       (net 5 "Net-(D2-DOUT)") (pinfunction "DIN") (pintype "input"))
     (model "${KICAD7_3DMODEL_DIR}/LED_SMD.3dshapes/LED_WS2812B_PLCC4_5.0x5.0mm_P3.2mm.wrl"
@@
   )
   (footprint "LED_SMD:LED_WS2812B_PLCC4_5.0x5.0mm_P3.2mm" (layer "F.Cu")
-    (at 177.8 63.5 180)
+    (at 177.8 63.5)
     (descr "5.0mm x 5.0mm Addressable RGB LED NeoPixel, https://cdn-shop.adafruit.com/datasheets/WS2812B.pdf")
     (tags "LED RGB NeoPixel PLCC-4 5050")
@@
     (fp_circle (center 0 0) (end 0 -2)
       (stroke (width 0.1) (type solid)) (fill none) (layer "F.Fab"))
-    (pad "1" smd rect (at -2.45 -1.65 180) (size 1.5 0.9) (layers "F.Cu" "F.Paste" "F.Mask")
+    (pad "1" smd rect (at -2.45 -1.65) (size 1.5 0.9) (layers "F.Cu" "F.Paste" "F.Mask")
       (net 1 "GND") (pinfunction "VDD") (pintype "power_in"))
-    (pad "2" smd rect (at -2.45 1.65 180) (size 1.5 0.9) (layers "F.Cu" "F.Paste" "F.Mask")
+    (pad "2" smd rect (at -2.45 1.65) (size 1.5 0.9) (layers "F.Cu" "F.Paste" "F.Mask")
       (net 3 "Net-(D1-DOUT)") (pinfunction "DOUT") (pintype "output"))
-    (pad "3" smd rect (at 2.45 1.65 180) (size 1.5 0.9) (layers "F.Cu" "F.Paste" "F.Mask")
+    (pad "3" smd rect (at 2.45 1.65) (size 1.5 0.9) (layers "F.Cu" "F.Paste" "F.Mask")
       (net 2 "Net-(D1-VSS)") (pinfunction "VSS") (pintype "power_in"))
-    (pad "4" smd rect (at 2.45 -1.65 180) (size 1.5 0.9) (layers "F.Cu" "F.Paste" "F.Mask")
+    (pad "4" smd rect (at 2.45 -1.65) (size 1.5 0.9) (layers "F.Cu" "F.Paste" "F.Mask")
       (net 4 "Net-(D1-DIN)") (pinfunction "DIN") (pintype "input"))
     (model "${KICAD7_3DMODEL_DIR}/LED_SMD.3dshapes/LED_WS2812B_PLCC4_5.0x5.0mm_P3.2mm.wrl"
@@
   )
   (footprint "LED_SMD:LED_WS2812B_PLCC4_5.0x5.0mm_P3.2mm" (layer "F.Cu")
-    (at 193.04 78.74 90)
+    (at 193.04 78.74)
     (descr "5.0mm x 5.0mm Addressable RGB LED NeoPixel, https://cdn-shop.adafruit.com/datasheets/WS2812B.pdf")
     (tags "LED RGB NeoPixel PLCC-4 5050")
@@
     (property "ki_keywords" "RGB LED NeoPixel addressable")
     (attr smd)
-    (fp_text reference "D2" (at 0 -3.5 90) (layer "F.SilkS")
-        (effects (font (size 1 1) (thickness 0.15)))
-    )
-    (fp_text value "WS2812B" (at 0 4 90) (layer "F.Fab")
-        (effects (font (size 1 1) (thickness 0.15)))
-    )
-    (fp_text user "1" (at -4.15 -1.6 90) (layer "F.SilkS")
-        (effects (font (size 1 1) (thickness 0.15)))
-    )
-    (fp_text user "${REFERENCE}" (at 0 0 90) (layer "F.Fab")
+    (fp_text reference "D2" (at 0 -3.5) (layer "F.SilkS")
+        (effects (font (size 1 1) (thickness 0.15)))
+    )
+    (fp_text value "WS2812B" (at 0 4) (layer "F.Fab")
+        (effects (font (size 1 1) (thickness 0.15)))
+    )
+    (fp_text user "1" (at -4.15 -1.6) (layer "F.SilkS")
+        (effects (font (size 1 1) (thickness 0.15)))
+    )
+    (fp_text user "${REFERENCE}" (at 0 0) (layer "F.Fab")
         (effects (font (size 0.8 0.8) (thickness 0.15)))
     )
@@
     (fp_circle (center 0 0) (end 0 -2)
       (stroke (width 0.1) (type solid)) (fill none) (layer "F.Fab"))
-    (pad "1" smd rect (at -2.45 -1.65 90) (size 1.5 0.9) (layers "F.Cu" "F.Paste" "F.Mask")
+    (pad "1" smd rect (at -2.45 -1.65) (size 1.5 0.9) (layers "F.Cu" "F.Paste" "F.Mask")
       (net 1 "GND") (pinfunction "VDD") (pintype "power_in"))
-    (pad "2" smd rect (at -2.45 1.65 90) (size 1.5 0.9) (layers "F.Cu" "F.Paste" "F.Mask")
+    (pad "2" smd rect (at -2.45 1.65) (size 1.5 0.9) (layers "F.Cu" "F.Paste" "F.Mask")
       (net 5 "Net-(D2-DOUT)") (pinfunction "DOUT") (pintype "output"))
-    (pad "3" smd rect (at 2.45 1.65 90) (size 1.5 0.9) (layers "F.Cu" "F.Paste" "F.Mask")
+    (pad "3" smd rect (at 2.45 1.65) (size 1.5 0.9) (layers "F.Cu" "F.Paste" "F.Mask")
       (net 2 "Net-(D1-VSS)") (pinfunction "VSS") (pintype "power_in"))
-    (pad "4" smd rect (at 2.45 -1.65 90) (size 1.5 0.9) (layers "F.Cu" "F.Paste" "F.Mask")
+    (pad "4" smd rect (at 2.45 -1.65) (size 1.5 0.9) (layers "F.Cu" "F.Paste" "F.Mask")
       (net 3 "Net-(D1-DOUT)") (pinfunction "DIN") (pintype "input"))
     (model "${KICAD7_3DMODEL_DIR}/LED_SMD.3dshapes/LED_WS2812B_PLCC4_5.0x5.0mm_P3.2mm.wrl"
@@
   (gr_rect (start 127 50.8) (end 203.2 127)
     (stroke (width 0.1) (type default)) (fill none) (layer "Edge.Cuts"))
-  (segment (start 172.08 63.5) (end 170.18 65.4) (width 0.25) (layer "F.Cu") (net 1))
   (segment (start 167.64 76.225) (end 174.786778 76.225) (width 0.25) (layer "F.Cu") (net 1))
-  (segment (start 180.25 65.15) (end 178.6 63.5) (width 0.25) (layer "F.Cu") (net 1))
   (segment (start 165.635 90.16) (end 162.835 90.16) (width 0.25) (layer "F.Cu") (net 1))
   (segment (start 162.835 91.56) (end 165.635 91.56) (width 0.25) (layer "F.Cu") (net 1))
@@
   (segment (start 174.86 76.298222) (end 174.86 83.465) (width 0.25) (layer "F.Cu") (net 1))
   (segment (start 162.835 88.69) (end 162.835 90.16) (width 0.25) (layer "F.Cu") (net 1))
-  (segment (start 178.6 63.5) (end 172.08 63.5) (width 0.25) (layer "F.Cu") (net 1))
   (segment (start 174.485 83.84) (end 171.955 83.84) (width 0.25) (layer "F.Cu") (net 1))
   (segment (start 174.786778 76.225) (end 174.86 76.298222) (width 0.25) (layer "F.Cu") (net 1))
@@
   (segment (start 165.635 92.96) (end 162.835 92.96) (width 0.25) (layer "F.Cu") (net 1))
   (segment (start 162.835 90.16) (end 162.835 91.56) (width 0.25) (layer "F.Cu") (net 1))
-  (segment (start 170.18 65.4) (end 167.64 67.94) (width 0.25) (layer "F.Cu") (net 1))
-  (segment (start 170.18 63.5) (end 171.83 61.85) (width 0.25) (layer "F.Cu") (net 2))
-  (segment (start 171.83 61.85) (end 175.35 61.85) (width 0.25) (layer "F.Cu") (net 2))
-  (segment (start 177.8 67.6) (end 175.35 65.15) (width 0.25) (layer "F.Cu") (net 4))
-  (segment (start 177.8 70.2075) (end 177.8 67.6) (width 0.25) (layer "F.Cu") (net 4))
   (segment (start 177.8 72.0325) (end 177.8 82.795) (width 0.25) (layer "F.Cu") (net 14))
   (segment (start 177.8 82.795) (end 175.485 85.11) (width 0.25) (layer "F.Cu") (net 14))
