File: KiCad/EntangledHearts/EntangledHearts.kicad_sch (KiCad schematic)
At the start: 56 parts

Commit message: ADD: further progress
Parts:
- added GND1: GND1, TestPoint:TestPoint_Pad_1.5x1.5mm, symbol Connector:TestPoint
- added GND2: GND2, TestPoint:TestPoint_Pad_1.5x1.5mm, symbol Connector:TestPoint
- added NeoPixel1: NeoPixel1, TestPoint:TestPoint_Pad_1.5x1.5mm, symbol Connector:TestPoint
- added NeoPixel2: NeoPixel2, TestPoint:TestPoint_Pad_1.5x1.5mm, symbol Connector:TestPoint
- added SCL1: SCL1, TestPoint:TestPoint_Pad_1.5x1.5mm, symbol Connector:TestPoint
- added SCL2: SCL2, TestPoint:TestPoint_Pad_1.5x1.5mm, symbol Connector:TestPoint
- added SDA1: SDA1, TestPoint:TestPoint_Pad_1.5x1.5mm, symbol Connector:TestPoint
- added SDA2: SDA2, TestPoint:TestPoint_Pad_1.5x1.5mm, symbol Connector:TestPoint
- added VCC1: VCC1, TestPoint:TestPoint_Pad_1.5x1.5mm, symbol Connector:TestPoint
- added VCC2: VCC2, TestPoint:TestPoint_Pad_1.5x1.5mm, symbol Connector:TestPoint
Connections:
- net +3.3V: now also PU_Photo1.2
- net +4V: now also VCC1.1; no longer C_NP1.1, C_NP2.1, C_NP3.1, C_NP4.1, C_NP5.1, C_NP6.1, D1.1 (VDD), D2.1 (VDD), D3.1 (VDD), D4.1 (VDD), D5.1 (VDD), D6.1 (VDD), Display1.3 (Pin_3)
- net GND: now also GND1.1; no longer C_NP1.2, C_NP2.2, C_NP3.2, C_NP4.2, C_NP5.2, C_NP6.2, D1.3 (VSS), D2.3 (VSS), D3.3 (VSS), D4.3 (VSS), D5.3 (VSS), D6.3 (VSS), Display1.4 (Pin_4)
- net at ButtonB2.1: now also Button1.2; no longer Button1.3
- net NeoPixel renamed NeoPixelBottom
- net NeoPixelBottom: no longer R_NP1.1
- net SCL renamed SCL_Bottom
- net SCL_Bottom: now also ESP1.20 (GPIO12/TOUCH12/ADC2_CH1/FSPICLK/FSPIIO6/SUBSPICLK), SCL1.1; no longer Display1.2 (Pin_2), ESP1.19 (GPIO11/TOUCH11/ADC2_CH0/FSPID/FSPIIO5/SUBSPID)
- net SDA renamed SDA_Bottom
- net SDA_Bottom: now also ESP1.19 (GPIO11/TOUCH11/ADC2_CH0/FSPID/FSPIIO5/SUBSPID), SDA1.1; no longer Display1.1 (Pin_1), ESP1.20 (GPIO12/TOUCH12/ADC2_CH1/FSPICLK/FSPIIO6/SUBSPICLK)
- new net GND_Top: C_NP1.2, C_NP2.2, C_NP3.2, C_NP4.2, C_NP5.2, C_NP6.2, D1.3 (VSS), D2.3 (VSS), D3.3 (VSS), D4.3 (VSS), D5.3 (VSS), D6.3 (VSS), Display1.4 (Pin_4), GND2.1
- new net NeoPixel_Bottom: NeoPixel1.1
- new net NeoPixel_Top: NeoPixel2.1, R_NP1.1
- new net SCL_Top: Display1.2 (Pin_2), SCL2.1
- new net SDA_Top: Display1.1 (Pin_1), SDA2.1
- new net VCC_Top: C_NP1.1, C_NP2.1, C_NP3.1, C_NP4.1, C_NP5.1, C_NP6.1, D1.1 (VDD), D2.1 (VDD), D3.1 (VDD), D4.1 (VDD), D5.1 (VDD), D6.1 (VDD), Display1.3 (Pin_3), VCC2.1
Other:
- moved on the sheet: ButtonB2, Display1, MPU1, PU_SCL1, PU_SDA1

Commit message: CHG: some minor changes
Parts:
- R_NP1: value 300Ω -> 330Ω
Connections:
- net +4V: no longer MPU1.1 (Pin_1)
- net GND: no longer MPU1.2 (Pin_2)
- net GND_Top: now also MPU1.2 (Pin_2)
- net SCL_Bottom: no longer MPU1.3 (Pin_3)
- net SCL_Top: now also MPU1.3 (Pin_3)
- net SDA_Bottom: no longer MPU1.4 (Pin_4)
- net SDA_Top: now also MPU1.4 (Pin_4)
- net VCC_Top: now also MPU1.1 (Pin_1)
Changed lines of the file:
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@@
     (stroke (width 0) (type default))
   )
-  (wire (pts (xy 257.81 200.66) (xy 265.43 200.66))
-    (stroke (width 0) (type default))
-  )
   (wire (pts (xy 378.46 139.7) (xy 381 139.7))
     (stroke (width 0) (type default))
@@
     (stroke (width 0) (type default))
   )
-  (wire (pts (xy 260.35 205.74) (xy 260.35 210.82))
+  (wire (pts (xy 123.19 241.3) (xy 138.43 241.3))
     (stroke (width 0) (type default))
   )
-  (wire (pts (xy 123.19 241.3) (xy 138.43 241.3))
+  (wire (pts (xy 265.43 207.01) (xy 265.43 210.82))
     (stroke (width 0) (type default))
   )
@@
     (stroke (width 0) (type default))
   )
-  (wire (pts (xy 262.89 203.2) (xy 262.89 210.82))
-    (stroke (width 0) (type default))
-  )
   (wire (pts (xy 339.09 189.23) (xy 351.79 189.23))
     (stroke (width 0) (type default))
@@
     (stroke (width 0) (type default))
   )
-  (wire (pts (xy 257.81 205.74) (xy 260.35 205.74))
-    (stroke (width 0) (type default))
-  )
   (wire (pts (xy 345.44 208.28) (xy 345.44 186.69))
     (stroke (width 0) (type default))
@@
     (stroke (width 0) (type default))
   )
-  (wire (pts (xy 257.81 198.12) (xy 267.97 198.12))
-    (stroke (width 0) (type default))
-  )
   (wire (pts (xy 161.29 83.82) (xy 168.91 83.82))
     (stroke (width 0) (type default))
@@
     (stroke (width 0) (type default))
   )
-  (wire (pts (xy 257.81 203.2) (xy 262.89 203.2))
-    (stroke (width 0) (type default))
-  )
   (wire (pts (xy 208.28 257.81) (xy 227.33 257.81))
     (stroke (width 0) (type default))
@@
     (stroke (width 0) (type default))
   )
-  (wire (pts (xy 265.43 200.66) (xy 265.43 210.82))
-    (stroke (width 0) (type default))
-  )
   (wire (pts (xy 342.9 129.54) (xy 345.44 129.54))
     (stroke (width 0) (type default))
@@
     (stroke (width 0) (type default))
   )
+  (wire (pts (xy 267.97 207.01) (xy 267.97 210.82))
+    (stroke (width 0) (type default))
+  )
   (wire (pts (xy 64.77 80.01) (xy 69.85 80.01))
     (stroke (width 0) (type default))
@@
     (stroke (width 0) (type default))
   )
-  (wire (pts (xy 156.21 41.91) (xy 156.21 38.1))
+  (wire (pts (xy 260.35 207.01) (xy 260.35 210.82))
     (stroke (width 0) (type default))
   )
-  (wire (pts (xy 157.48 226.06) (xy 157.48 236.22))
+  (wire (pts (xy 156.21 41.91) (xy 156.21 38.1))
     (stroke (width 0) (type default))
   )
-  (wire (pts (xy 267.97 198.12) (xy 267.97 210.82))
+  (wire (pts (xy 157.48 226.06) (xy 157.48 236.22))
     (stroke (width 0) (type default))
   )
@@
     (stroke (width 0) (type default))
   )
+  (wire (pts (xy 262.89 207.01) (xy 262.89 210.82))
+    (stroke (width 0) (type default))
+  )
   (wire (pts (xy 62.23 243.84) (xy 74.93 243.84))
     (stroke (width 0) (type default))
@@
     )
   )
+  (global_label "SCL_Top" (shape input) (at 265.43 207.01 90) (fields_autoplaced)
+    (effects (font (size 1.27 1.27)) (justify left))
+    (property "Intersheetrefs" "${INTERSHEET_REFS}" (at 265.43 196.284 90)
+      (effects (font (size 1.27 1.27)) (justify left) hide)
+    )
+  )
   (global_label "GND" (shape input) (at 205.74 163.83 180) (fields_autoplaced)
     (effects (font (size 1.27 1.27)) (justify right))
@@
     )
   )
+  (global_label "VCC_Top" (shape input) (at 260.35 207.01 90) (fields_autoplaced)
+    (effects (font (size 1.27 1.27)) (justify left))
+    (property "Intersheetrefs" "${INTERSHEET_REFS}" (at 260.35 196.163 90)
+      (effects (font (size 1.27 1.27)) (justify left) hide)
+    )
+  )
   (global_label "RXD" (shape input) (at 341.63 160.02 0) (fields_autoplaced)
     (effects (font (size 1.27 1.27)) (justify left))
@@
     )
   )
-  (global_label "SCL_Bottom" (shape input) (at 257.81 200.66 180) (fields_autoplaced)
-    (effects (font (size 1.27 1.27)) (justify right))
-    (property "Intersheetrefs" "${INTERSHEET_REFS}" (at 243.6369 200.66 0)
-      (effects (font (size 1.27 1.27)) (justify right) hide)
-    )
-  )
   (global_label "TXD" (shape input) (at 262.89 86.36 0) (fields_autoplaced)
     (effects (font (size 1.27 1.27)) (justify left))
@@
     )
   )
+  (global_label "GND_Top" (shape input) (at 262.89 207.01 90) (fields_autoplaced)
+    (effects (font (size 1.27 1.27)) (justify left))
+    (property "Intersheetrefs" "${INTERSHEET_REFS}" (at 262.89 195.9211 90)
+      (effects (font (size 1.27 1.27)) (justify left) hide)
+    )
+  )
+  (global_label "SDA_Top" (shape input) (at 267.97 207.01 90) (fields_autoplaced)
+    (effects (font (size 1.27 1.27)) (justify left))
+    (property "Intersheetrefs" "${INTERSHEET_REFS}" (at 267.97 196.2235 90)
+      (effects (font (size 1.27 1.27)) (justify left) hide)
+    )
+  )
   (global_label "GND_Top" (shape input) (at 309.88 26.67 0) (fields_autoplaced)
     (effects (font (size 1.27 1.27)) (justify left))
@@
     )
   )
-  (global_label "SDA_Bottom" (shape input) (at 257.81 198.12 180) (fields_autoplaced)
-    (effects (font (size 1.27 1.27)) (justify right))
-    (property "Intersheetrefs" "${INTERSHEET_REFS}" (at 243.5764 198.12 0)
-      (effects (font (size 1.27 1.27)) (justify right) hide)
-    )
-  )
   (global_label "Boot" (shape input) (at 297.18 99.06 0) (fields_autoplaced)
     (effects (font (size 1.27 1.27)) (justify left))
@@
     )
   )
-  (symbol (lib_id "power:+4V") (at 257.81 205.74 90) (unit 1)
-    (in_bom yes) (on_board yes) (dnp no) (fields_autoplaced)
-    (property "Reference" "#PWR016" (at 261.62 205.74 0)
-      (effects (font (size 1.27 1.27)) hide)
-    )
-    (property "Value" "+4V" (at 254 205.74 90)
-      (effects (font (size 1.27 1.27)) (justify left))
-    )
-    (property "Footprint" "" (at 257.81 205.74 0)
-      (effects (font (size 1.27 1.27)) hide)
-    )
-    (property "Datasheet" "" (at 257.81 205.74 0)
-      (effects (font (size 1.27 1.27)) hide)
-    )
-    (pin "1")
-    (instances
-      (project "EntangledHearts"
-        (path "/13d221e6-7345-4ae4-985d-7c8e9051407d"
-          (reference "#PWR016") (unit 1)
-        )
-      )
-    )
-  )
   (symbol (lib_id "USB4135-GF-A:USB4135-GF-A") (at 62.23 233.68 0) (mirror y) (unit 1)
     (in_bom yes) (on_board yes) (dnp no)
@@
     )
   )
-  (symbol (lib_id "power:GND") (at 257.81 203.2 270) (unit 1)
-    (in_bom yes) (on_board yes) (dnp no) (fields_autoplaced)
-    (property "Reference" "#PWR017" (at 251.46 203.2 0)
-      (effects (font (size 1.27 1.27)) hide)
-    )
-    (property "Value" "GND" (at 254 203.2 90)
-      (effects (font (size 1.27 1.27)) (justify right))
-    )
-    (property "Footprint" "" (at 257.81 203.2 0)
-      (effects (font (size 1.27 1.27)) hide)
-    )
-    (property "Datasheet" "" (at 257.81 203.2 0)
-      (effects (font (size 1.27 1.27)) hide)
-    )
-    (pin "1")
-    (instances
-      (project "EntangledHearts"
-        (path "/13d221e6-7345-4ae4-985d-7c8e9051407d"
-          (reference "#PWR017") (unit 1)
-        )
-      )
-    )
-  )
   (symbol (lib_id "LED:WS2812B") (at 245.11 34.29 180) (unit 1)
     (in_bom yes) (on_board yes) (dnp no)
@@
       (effects (font (size 1.27 1.27)))
     )
-    (property "Value" "300Ω" (at 295.91 30.48 90)
+    (property "Value" "330Ω" (at 295.91 30.48 90)
       (effects (font (size 1.27 1.27)))
     )

Commit message: ADD: all parts connected
Parts:
- removed +Bat1: + Bat, TestPoint:TestPoint_Pad_2.5x2.5mm, symbol Connector:TestPoint
- removed -Bat1: - Bat, TestPoint:TestPoint_Pad_2.5x2.5mm, symbol Connector:TestPoint
- added BatteryConnector1: BatteryConnector, Connector_JST:JST_PH_S2B-PH-SM4-TB_1x02-1MP_P2.00mm_Horizontal, symbol Connector_Generic:Conn_01x02
- renumbered PM1 to BM1, BM1 to PM1
Connections:
- net GND: now also BatteryConnector1.1 (Pin_1)
- net NeoPixel_Bottom: now also ESP1.11 (GPIO18/U1RXD/ADC2_CH7/CLK_OUT3)
- net at BM1.3 (V_{BAT}), CP2.1, CP3.1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: now also BatteryConnector1.2 (Pin_2)
- net NeoPixelBottom: no longer names the net of ESP1.23 (GPIO21)
Changed lines of the file:
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@@
   (junction (at 69.85 80.01) (diameter 0) (color 0 0 0 0)
   )
+  (junction (at 147.32 257.81) (diameter 0) (color 0 0 0 0)
+  )
   (junction (at 170.18 257.81) (diameter 0) (color 0 0 0 0)
   )
   (junction (at 232.41 26.67) (diameter 0) (color 0 0 0 0)
   )
-  (junction (at 144.78 257.81) (diameter 0) (color 0 0 0 0)
-  )
   (junction (at 195.58 257.81) (diameter 0) (color 0 0 0 0)
   )
@@
   (junction (at 36.83 238.76) (diameter 0) (color 0 0 0 0)
   )
-  (junction (at 260.35 142.24) (diameter 0) (color 0 0 0 0)
-  )
   (junction (at 274.32 114.3) (diameter 0) (color 0 0 0 0)
   )
@@
     (stroke (width 0) (type default))
   )
-  (wire (pts (xy 260.35 142.24) (xy 264.16 142.24))
-    (stroke (width 0) (type default))
-  )
   (wire (pts (xy 260.35 83.82) (xy 262.89 83.82))
     (stroke (width 0) (type default))
@@
     (stroke (width 0) (type default))
   )
+  (wire (pts (xy 260.35 139.7) (xy 264.16 139.7))
+    (stroke (width 0) (type default))
+  )
   (wire (pts (xy 149.86 257.81) (xy 170.18 257.81))
     (stroke (width 0) (type default))
@@
     (stroke (width 0) (type default))
   )
-  (wire (pts (xy 144.78 257.81) (xy 149.86 257.81))
-    (stroke (width 0) (type default))
-  )
   (wire (pts (xy 181.61 41.91) (xy 181.61 38.1))
     (stroke (width 0) (type default))
@@
     (stroke (width 0) (type default))
   )
-  (wire (pts (xy 144.78 207.01) (xy 144.78 257.81))
+  (wire (pts (xy 147.32 207.01) (xy 147.32 257.81))
     (stroke (width 0) (type default))
   )
@@
     (stroke (width 0) (type default))
   )
-  (wire (pts (xy 342.9 129.54) (xy 345.44 129.54))
-    (stroke (width 0) (type default))
-  )
   (wire (pts (xy 157.48 238.76) (xy 157.48 236.22))
     (stroke (width 0) (type default))
@@
     (stroke (width 0) (type default))
   )
-  (wire (pts (xy 125.73 257.81) (xy 144.78 257.81))
+  (wire (pts (xy 125.73 257.81) (xy 147.32 257.81))
     (stroke (width 0) (type default))
   )
@@
     (stroke (width 0) (type default))
   )
+  (wire (pts (xy 342.9 129.54) (xy 345.44 129.54))
+    (stroke (width 0) (type default))
+  )
   (wire (pts (xy 81.28 242.57) (xy 81.28 257.81))
     (stroke (width 0) (type default))
@@
     (stroke (width 0) (type default))
   )
+  (wire (pts (xy 147.32 257.81) (xy 149.86 257.81))
+    (stroke (width 0) (type default))
+  )
   (wire (pts (xy 36.83 257.81) (xy 68.58 257.81))
     (stroke (width 0) (type default))
@@
     )
   )
-  (global_label "NeoPixelBottom" (shape input) (at 264.16 142.24 0) (fields_autoplaced)
+  (global_label "NeoPixel_Bottom" (shape input) (at 264.16 139.7 0) (fields_autoplaced)
     (effects (font (size 1.27 1.27)) (justify left))
-    (property "Intersheetrefs" "${INTERSHEET_REFS}" (at 282.0827 142.24 0)
+    (property "Intersheetrefs" "${INTERSHEET_REFS}" (at 283.0503 139.7 0)
       (effects (font (size 1.27 1.27)) (justify left) hide)
     )
@@
   (symbol (lib_id "Regulator_Linear:TC1185-xCT") (at 170.18 238.76 0) (unit 1)
     (in_bom yes) (on_board yes) (dnp no) (fields_autoplaced)
-    (property "Reference" "BM1" (at 170.18 228.6 0)
+    (property "Reference" "PM1" (at 170.18 228.6 0)
       (effects (font (size 1.27 1.27)))
     )
@@
       (project "EntangledHearts"
         (path "/13d221e6-7345-4ae4-985d-7c8e9051407d"
-          (reference "BM1") (unit 1)
+          (reference "PM1") (unit 1)
         )
       )
@@
   (symbol (lib_id "Battery_Management:MCP73831-2-OT") (at 113.03 238.76 0) (unit 1)
     (in_bom yes) (on_board yes) (dnp no) (fields_autoplaced)
-    (property "Reference" "PM1" (at 115.2241 228.6 0)
+    (property "Reference" "BM1" (at 115.2241 228.6 0)
       (effects (font (size 1.27 1.27)) (justify left))
     )
@@
       (project "EntangledHearts"
         (path "/13d221e6-7345-4ae4-985d-7c8e9051407d"
-          (reference "PM1") (unit 1)
+          (reference "BM1") (unit 1)
         )
       )
@@
     )
   )
-  (symbol (lib_id "Connector:TestPoint") (at 149.86 207.01 0) (mirror y) (unit 1)
-    (in_bom yes) (on_board yes) (dnp no)
-    (property "Reference" "+Bat1" (at 153.67 198.12 0)
-      (effects (font (size 1.27 1.27)) (justify left))
-    )
-    (property "Value" "+ Bat" (at 153.67 200.66 0)
-      (effects (font (size 1.27 1.27)) (justify left))
-    )
-    (property "Footprint" "TestPoint:TestPoint_Pad_2.5x2.5mm" (at 144.78 207.01 0)
-      (effects (font (size 1.27 1.27)) hide)
-    )
-    (property "Datasheet" "~" (at 144.78 207.01 0)
-      (effects (font (size 1.27 1.27)) hide)
-    )
-    (pin "1")
-    (instances
-      (project "EntangledHearts"
-        (path "/13d221e6-7345-4ae4-985d-7c8e9051407d"
-          (reference "+Bat1") (unit 1)
-        )
-      )
-    )
-  )
   (symbol (lib_id "LED:WS2812B") (at 143.51 34.29 180) (unit 1)
     (in_bom yes) (on_board yes) (dnp no)
@@
     )
   )
-  (symbol (lib_id "Connector:TestPoint") (at 144.78 207.01 0) (mirror y) (unit 1)
-    (in_bom yes) (on_board yes) (dnp no)
-    (property "Reference" "-Bat1" (at 146.05 198.12 0)
-      (effects (font (size 1.27 1.27)) (justify left))
-    )
-    (property "Value" "- Bat" (at 146.05 200.66 0)
-      (effects (font (size 1.27 1.27)) (justify left))
-    )
-    (property "Footprint" "TestPoint:TestPoint_Pad_2.5x2.5mm" (at 139.7 207.01 0)
-      (effects (font (size 1.27 1.27)) hide)
-    )
-    (property "Datasheet" "~" (at 139.7 207.01 0)
-      (effects (font (size 1.27 1.27)) hide)
-    )
-    (pin "1")
-    (instances
-      (project "EntangledHearts"
-        (path "/13d221e6-7345-4ae4-985d-7c8e9051407d"
-          (reference "-Bat1") (unit 1)
-        )
-      )
-    )
-  )
   (symbol (lib_id "Device:C") (at 125.73 251.46 0) (unit 1)
     (in_bom yes) (on_board yes) (dnp no) (fields_autoplaced)
@@
         )
       )
+    )
+  )
+  (symbol (lib_id "Connector_Generic:Conn_01x02") (at 147.32 201.93 90) (unit 1)
+    (in_bom yes) (on_board yes) (dnp no)
+    (property "Reference" "BatteryConnector1" (at 139.7 196.85 90)
+      (effects (font (size 1.27 1.27)) (justify right))
+    )
+    (property "Value" "BatteryConnector" (at 139.7 199.39 90)
+      (effects (font (size 1.27 1.27)) (justify right))
+    )
+    (property "Footprint" "Connector_JST:JST_PH_S2B-PH-SM4-TB_1x02-1MP_P2.00mm_Horizontal" (at 147.32 201.93 0)
+      (effects (font (size 1.27 1.27)) hide)
+    )
+    (property "Datasheet" "~" (at 147.32 201.93 0)
+      (effects (font (size 1.27 1.27)) hide)
+    )
+    (pin "2")
+    (pin "1")
+    (instances
+      (project "EntangledHearts"
+        (path "/13d221e6-7345-4ae4-985d-7c8e9051407d"
+          (reference "BatteryConnector1") (unit 1)
+        )
+      )

Commit message: ADD: all components connected
Connections:
- net Button: now also ESP1.6 (GPIO6/TOUCH6/ADC1_CH5); no longer ESP1.39 (GPIO1/TOUCH1/ADC1_CH0)
Changed lines of the file:
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@@
-    (stroke (width 0) (type default))
-  )
-  (wire (pts (xy 260.35 101.6) (xy 262.89 101.6))
     (stroke (width 0) (type default))
   )
@@
   )
   (wire (pts (xy 157.48 238.76) (xy 157.48 236.22))
+    (stroke (width 0) (type default))
+  )
+  (wire (pts (xy 260.35 114.3) (xy 262.89 114.3))
     (stroke (width 0) (type default))
   )
@@
   )
   (text_box "internal PullUp"
-    (at 271.78 100.33 0) (size 16.51 2.54)
+    (at 260.35 110.49 0) (size 16.51 2.54)
     (stroke (width 0) (type default))
     (fill (type none))
@@
     )
   )
-  (global_label "Button" (shape input) (at 262.89 101.6 0) (fields_autoplaced)
-    (effects (font (size 1.27 1.27)) (justify left))
-    (property "Intersheetrefs" "${INTERSHEET_REFS}" (at 272.0436 101.6 0)
-      (effects (font (size 1.27 1.27)) (justify left) hide)
-    )
+  (global_label "Button" (shape input) (at 262.89 114.3 0) (fields_autoplaced)
+    (effects (font (size 1.27 1.27)) (justify left))
+    (property "Intersheetrefs" "${INTERSHEET_REFS}" (at 272.0436 114.3 0)
+      (effects (font (size 1.27 1.27)) (justify left) hide)
+    )
